File: hardware/8bit_hex_display.kicad_sch (KiCad schematic)
At the start: 28 parts, among them U1 74HC163, U2 74HC163, U3 74HC10, U4 DA04-11SRWA, U5 74LS47, U6 74LS47

Commit message: Episode 2
Parts:
- removed C6: 100n, symbol Device:C_Small
- removed R1, R10, R11, R12, R13, R14, R2, R3, R4, R5, R6, R7, R8, R9: 280, symbol Device:R_Small
- removed U3: 74HC10, symbol 74xx:74LS10
- removed U4: DA04-11SRWA, Display_7Segment:DA04-11SURKWA, symbol Display_Character:DA04-11SRWA
- removed U5, U6: 74LS47, symbol 74xx:74LS47
- added U4, U6: MC14495, Package_DIP:DIP-16_W7.62mm, symbol 8bit_hex_display:MC14495
- added U5: HDSP-523Y, Display_7Segment:DA56-11SYKWA, symbol Display_Character:DC56-11YWA
Connections:
- net D0: now also U6.5 (A)
- net D1: now also U6.6 (B)
- net D2: now also U6.9 (C)
- net D3: now also U6.10 (D)
- net D4: now also U4.5 (A)
- net D5: now also U4.6 (B)
- net D6: now also U4.9 (C)
- net D7: now also U4.10 (D)
- net GND: now also U4.8 (GND), U5.13 (DIG2_CC), U5.14 (DIG1_CC), U6.8 (GND)
- net VCC: now also U1.1 (~{MR}), U2.1 (~{MR}), U4.16 (VCC), U6.16 (VCC)
- net at U2.10 (CET): now also U1.15 (TC)
- new net: U5.5 (DIG2_E), U6.1 (e)
- new net: U5.11 (DIG2_A), U6.12 (a)
- new net: U5.10 (DIG2_B), U6.13 (b)
- new net: U5.8 (DIG2_C), U6.14 (c)
- new net: U5.6 (DIG2_D), U6.15 (d)
- new net: U5.12 (DIG2_F), U6.2 (f)
- new net: U5.7 (DIG2_G), U6.3 (g)
- new net: U4.1 (e), U5.1 (DIG1_E)
- new net: U4.12 (a), U5.16 (DIG1_A)
- new net: U4.13 (b), U5.15 (DIG1_B)
- new net: U4.14 (c), U5.3 (DIG1_C)
- new net: U4.15 (d), U5.2 (DIG1_D)
- new net: U4.2 (f), U5.18 (DIG1_F)
- new net: U4.3 (g), U5.17 (DIG1_G)
- new net LE: U4.7 (LE), U6.7 (LE)
- no-connect marks 2 -> 7
Other:
- note added: "MC14495: V(on) = -0.31*I + 4.71667 (linear regression) HDSP-523Y V_F = 0.025*I + 1.63333 (approx from graph, linear regression) => V(on) = V_F => -0.31*I + 4.717 = 0.025*I + 1.633 => 3.084 = 0.285*I => I = 10.82mA I_V = 2.3 mcd @ 10mA => I_V = 2.3 * 10.82 / 10 = 2.48 mcd"
- note removed: "74LS47 VO(on) @ 12mA is 0.25V typical, 0.4V maximum IO(on) is 24mA maximum At 10mA: DA04-11YWA (yellow): V_F is 1.95 typical, 2.4V maximum => R = (5V - 1.95V - 0.25V) / 10mA = 2.8V / 0.01A = 280 ohms DA04-11PBWA (blue): V_F is 3.1 typical (from graph) => R = (5V - 3.1V - 0.25V) / 10mA = 1.65V / 0.01A = 165 ohms DA04-11SRWA (red): V_F is 1.8 typical, 2.3V maximum => R = (5V - 1.8V - 0.25V) / 10mA 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"
